File: board/project/intellicart.kicad_pcb (KiCad board)
At the start: 2 copper layers, 68.1 x 90.1 mm, 22 parts, among them J1 2x22 card edge connector, J2 Oled 0.91" female, SW1 SW_Push, SW2 SW_Push, SW3 SW_Push, U1 74LS245, U2 74LS245, U3 74LVS45, U4 Teensy4.1, U5 74L245

Commit message: Refine r1.3 manufacturing draft
Parts:
- U1, U2: value 74LS245 -> 74LVC245
- U3: value 74LVS45 -> 74LVC245
- U5: value 74L245 -> 74LVC245
Other:
- outline, holes or cut-outs redrawn
- board text added: "GND"
- board text added: "INTELLICART"
- board text added: "cartheur"
- board text removed: "Intellicart from Cartheur Research v1.2"
- board text removed: "gnd"

Commit message: Make board profile standalone
Other:
- board size 68.1 x 90.1 mm -> 68.1 x 98.9 mm
Changed lines of the file:
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@@
 		(duplicate_pad_numbers_are_jumpers no)
-		(fp_line
-			(start 0 7.39)
-			(end 0 0)
-			(stroke
-				(width 0.12)
-				(type solid)
-			)
-			(layer "Edge.Cuts")
-		)
-		(fp_line
-			(start 0 7.39)
-			(end 1.45 8.84)
-			(stroke
-				(width 0.12)
-				(type solid)
-			)
-			(layer "Edge.Cuts")
-		)
-		(fp_line
-			(start 56.7414 8.84)
-			(end 1.45 8.84)
-			(stroke
-				(width 0.12)
-				(type solid)
-			)
-			(layer "Edge.Cuts")
-		)
-		(fp_line
-			(start 58.1914 7.39)
-			(end 56.7414 8.84)
-			(stroke
-				(width 0.12)
-				(type solid)
-			)
-			(layer "Edge.Cuts")
-		)
-		(fp_line
-			(start 58.1914 7.39)
-			(end 58.1914 0)
-			(stroke
-				(width 0.12)
-				(type solid)
-			)
-			(layer "Edge.Cuts")
-		)
 		(fp_line
 			(start 0 0)
@@
 	)
 	(gr_line
+		(start 88.9 190.93)
+		(end 88.9 183.54)
+		(stroke
+			(width 0.12)
+			(type solid)
+		)
+		(layer "Edge.Cuts")
+	)
+	(gr_line
+		(start 88.9 190.93)
+		(end 90.35 192.38)
+		(stroke
+			(width 0.12)
+			(type solid)
+		)
+		(layer "Edge.Cuts")
+	)
+	(gr_line
+		(start 145.6414 192.38)
+		(end 90.35 192.38)
+		(stroke
+			(width 0.12)
+			(type solid)
+		)
+		(layer "Edge.Cuts")
+	)
+	(gr_line
+		(start 147.0914 190.93)
+		(end 145.6414 192.38)
+		(stroke
+			(width 0.12)
+			(type solid)
+		)
+		(layer "Edge.Cuts")
+	)
+	(gr_line
+		(start 147.0914 190.93)
+		(end 147.0914 183.54)
+		(stroke
+			(width 0.12)
+			(type solid)
+		)
+		(layer "Edge.Cuts")
+	)
+	(gr_line
